File: KICAD/udb-sx.kicad_pcb (KiCad board)
At the start: 2 copper layers, 40 x 9 mm, 11 parts, among them J0 USB_C_Receptacle, J1 JST-SH-04, J2 JST-SUR-04, J3 Conn_01x04

Commit message: Update udb-sx.kicad_pcb
Parts:
- moved C1 1.50 mm to (100.0, 46.5)
- moved R3 1.50 mm to (100.0, 48.0)
- moved J2 0.08 mm to (90.5, 52.9)
Routing:
- net D-: track 34.9 -> 37.2 mm
- net VCC: track 27.4 -> 26.4 mm
- net GND: track 41.5 -> 42.5 mm, vias 10 -> 9
- net D+: track 35.1 -> 36.0 mm
- net VBUS: track 19.4 -> 18.5 mm
- net Net-(J0-CC1): track 12.6 -> 12.1 mm

Commit message: .
Parts:
- added C2: 1nF, Capacitor_SMD:C_0603_1608Metric, F.Cu at (100.0, 52.2)
- added FB1: 600Ω @ 100MHz, Inductor_SMD:L_0603_1608Metric, F.Cu at (100.0, 46.3)
- C1: value 4.7uF -> 0.1uF
- moved C1 7.20 mm to (100.0, 53.7)
- moved F1 3.57 mm to (95.8, 52.3), turned to 90 degrees
- moved R1 0.30 mm to (100.0, 49.2)
- moved R2 0.30 mm to (100.0, 50.7)
- moved R3 0.30 mm to (100.0, 47.7)
Routing:
- net GND: track 42.5 -> 33.8 mm, vias 9 -> 10
- net VBUS: track 18.5 -> 23.6 mm
- net VCC: track 26.4 -> 24.0 mm, vias 3 -> 2
Other:
- board text added: "Data"

Commit message: update
Parts:
- J1: footprint Connector_JST:JST_SH_SM04B-SRSS-TB_1x04-1MP_P1.00mm_Horizontal -> ts-keyboard-lib:JST_SH_SM04B-SRSS-TB_1x04-1MP_P1.00mm_Horizontal
Routing:
- net Earth: track 3.77 -> 0.14 mm, vias 1 -> 5
- net GND: track 33.8 -> 34.4 mm
