File: KICAD/udb-sx.kicad_sch (KiCad schematic)
At the start: 12 parts, among them J0 USB_C_Receptacle, J1 JST-SH-04, J2 JST-SUR-04, J3 Conn_01x04

Commit message: .
Parts:
- added C2: 1nF, Capacitor_SMD:C_0603_1608Metric, symbol Device:C
- added FB1: 600Ω @ 100MHz, Inductor_SMD:L_0603_1608Metric, symbol ts-kicad-lib:Ferrite_Bead
- C1: value 4.7uF -> 0.1uF
Connections:
- net Earth: now also C2.1, FB1.1
- net GND: now also C2.2, FB1.2
Other:
- moved on the sheet: R3

Commit message: update
Parts:
- J1: footprint Connector_JST:JST_SH_SM04B-SRSS-TB_1x04-1MP_P1.00mm_Horizontal -> ts-keyboard-lib:JST_SH_SM04B-SRSS-TB_1x04-1MP_P1.00mm_Horizontal
- R1, R2, R3: footprint Resistors_SMD:R_0603 -> Resistor_SMD:R_0603_1608Metric
- TVS1: symbol 1components:SP0503BAHTG -> 1:SP0503BAHTG
Connections:
- net Earth: now also J0.SH (SHIELD); no longer J0.S1 (SHIELD)
Other:
- moved on the sheet: F1
